File: can-bridge.kicad_sch (KiCad schematic)
At the start: 14 parts, among them J102 CAN1, SW101 78RB02ST, SW102 Reset, U102 MCP2551-I-SN, U104 TXB0104PW

Commit message: Added README.md and image of prototype
Changed R101 resistor to 1206 footprint
Parts:
- R101: footprint Resistor_SMD:R_0603_1608Metric -> Resistor_SMD:R_1206_3216Metric
Changed lines of the file:
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@@
 			)
 		)
-		(property "Footprint" "Resistor_SMD:R_0603_1608Metric"
+		(property "Footprint" "Resistor_SMD:R_1206_3216Metric"
 			(at 145.542 120.65 90)
 			(effects
